Commit message: Added position control

File: robot_arm/urdf/robot_arm.urdf.xacro (robot description, xacro)
@@ -487,4 +487,61 @@
           <param name="min">-1000.0</param>
           <param name="max">1000.0</param>
+        </command_interface>
+        <state_interface name="position"/>
+        <state_interface name="velocity"/>
+    </joint>
+    <!-- Position Controller -->
+    <joint name="ShoulderRollJoint">
+        <command_interface name="position">
+          <param name="min">-3.14</param>
+          <param name="max">3.14</param>
+        </command_interface>
+        <state_interface name="position"/>
+        <state_interface name="velocity"/>
+    </joint>
+    <joint name="ShoulderPitchJoint">
+        <command_interface name="position">
+          <param name="min">-3.14</param>
+          <param name="max">3.14</param>
+        </command_interface>
+        <state_interface name="position"/>
+        <state_interface name="velocity"/>
+    </joint>
+    <joint name="ArmRollJoint">
+        <command_interface name="position">
+          <param name="min">-3.14</param>
+          <param name="max">3.14</param>
+        </command_interface>
+        <state_interface name="position"/>
+        <state_interface name="velocity"/>
+    </joint>
+    <joint name="ElbowJoint">
+        <command_interface name="position">
+          <param name="min">-3.14</param>
+          <param name="max">3.14</param>
+        </command_interface>
+        <state_interface name="position"/>
+        <state_interface name="velocity"/>
+    </joint>
+    <joint name="WristRollJoint">
+        <command_interface name="position">
+          <param name="min">-3.14</param>
+          <param name="max">3.14</param>
+        </command_interface>
+        <state_interface name="position"/>
+        <state_interface name="velocity"/>
+    </joint>
+    <joint name="WristPitchJoint">
+        <command_interface name="position">
+          <param name="min">-3.14</param>
+          <param name="max">3.14</param>
+        </command_interface>
+        <state_interface name="position"/>
+        <state_interface name="velocity"/>
+    </joint>
+    <joint name="WristYawJoint">
+        <command_interface name="position">
+          <param name="min">-3.14</param>
+          <param name="max">3.14</param>
         </command_interface>
         <state_interface name="position"/>

Commit message: Combo works

File: robot_arm/urdf/robot_arm.urdf.xacro (robot description, xacro)
@@ -105,4 +105,5 @@
       xyz="0 0 -1" />
     <limit lower="-1.57" upper="1.57" effort="50" velocity="2.0" />
+    <dynamics damping="0.5" friction="0.1"/>
   </joint>
   <link
@@ -159,4 +160,5 @@
       xyz="0 0 -1" />
     <limit lower="-1.57" upper="1.57" effort="50" velocity="2.0" />
+    <dynamics damping="0.5" friction="0.1"/>
   </joint>
   <link
@@ -213,4 +215,5 @@
       xyz="0 0 -1" />
     <limit lower="-1.57" upper="1.57" effort="50" velocity="2.0" />
+    <dynamics damping="0.5" friction="0.1"/>
   </joint>
   <link
@@ -267,4 +270,5 @@
       xyz="0 0 -1" />
     <limit lower="-1.57" upper="1.57" effort="50" velocity="2.0" />
+    <dynamics damping="0.5" friction="0.1"/>
   </joint>
   <link
@@ -321,4 +325,5 @@
       xyz="0 0 1" />
     <limit lower="-1.57" upper="1.57" effort="50" velocity="2.0" />
+    <dynamics damping="0.5" friction="0.1"/>
   </joint>
   <link
@@ -375,4 +380,5 @@
       xyz="0 0 -1" />
     <limit lower="-1.57" upper="1.57" effort="50" velocity="2.0" />
+    <dynamics damping="0.5" friction="0.1"/>
   </joint>
   <link
@@ -429,4 +435,5 @@
       xyz="0 0 -1" />
     <limit lower="-1.57" upper="1.57" effort="50" velocity="2.0" />
+    <dynamics damping="0.5" friction="0.1"/>
   </joint>
   <ros2_control name="GazeboSystem" type="system">
@@ -497,3 +504,24 @@
     </plugin>
   </gazebo>
+  <gazebo reference="ShoulderRoll">
+   <turnGravityOff>true</turnGravityOff>
+  </gazebo>
+  <gazebo reference="ShoulderPitch">
+   <turnGravityOff>true</turnGravityOff>
+  </gazebo>
+  <gazebo reference="ArmRoll">
+   <turnGravityOff>true</turnGravityOff>
+  </gazebo>
+  <gazebo reference="Elbow">
+   <turnGravityOff>true</turnGravityOff>
+  </gazebo>
+  <gazebo reference="WristRoll">
+   <turnGravityOff>true</turnGravityOff>
+  </gazebo>
+  <gazebo reference="WristPitch">
+   <turnGravityOff>true</turnGravityOff>
+  </gazebo>
+  <gazebo reference="WristYaw">
+   <turnGravityOff>true</turnGravityOff>
+  </gazebo>
 </robot>

Commit message: Completed readme and prepared for submission

File: robot_arm/urdf/robot_arm.urdf.xacro (robot description, xacro)
@@ -105,5 +105,5 @@
       xyz="0 0 -1" />
     <limit lower="-1.57" upper="1.57" effort="50" velocity="2.0" />
-    <dynamics damping="0.5" friction="0.1"/>
+    <!-- <dynamics damping="0.5" friction="0.1"/> -->
   </joint>
   <link
@@ -160,5 +160,5 @@
       xyz="0 0 -1" />
     <limit lower="-1.57" upper="1.57" effort="50" velocity="2.0" />
-    <dynamics damping="0.5" friction="0.1"/>
+    <!-- <dynamics damping="0.5" friction="0.1"/> -->
   </joint>
   <link
@@ -215,5 +215,5 @@
       xyz="0 0 -1" />
     <limit lower="-1.57" upper="1.57" effort="50" velocity="2.0" />
-    <dynamics damping="0.5" friction="0.1"/>
+    <!-- <dynamics damping="0.5" friction="0.1"/> -->
   </joint>
   <link
@@ -270,5 +270,5 @@
       xyz="0 0 -1" />
     <limit lower="-1.57" upper="1.57" effort="50" velocity="2.0" />
-    <dynamics damping="0.5" friction="0.1"/>
+    <!-- <dynamics damping="0.5" friction="0.1"/> -->
   </joint>
   <link
@@ -325,5 +325,5 @@
       xyz="0 0 1" />
     <limit lower="-1.57" upper="1.57" effort="50" velocity="2.0" />
-    <dynamics damping="0.5" friction="0.1"/>
+    <!-- <dynamics damping="0.5" friction="0.1"/> -->
   </joint>
   <link
@@ -380,5 +380,5 @@
       xyz="0 0 -1" />
     <limit lower="-1.57" upper="1.57" effort="50" velocity="2.0" />
-    <dynamics damping="0.5" friction="0.1"/>
+    <!-- <dynamics damping="0.5" friction="0.1"/> -->
   </joint>
   <link
@@ -435,5 +435,5 @@
       xyz="0 0 -1" />
     <limit lower="-1.57" upper="1.57" effort="50" velocity="2.0" />
-    <dynamics damping="0.5" friction="0.1"/>
+    <!-- <dynamics damping="0.5" friction="0.1"/> -->
   </joint>
   <ros2_control name="GazeboSystem" type="system">
